Commit message: adicionando links e joints

File: AmbientesRos/simulation/src/my_robot_description/urdf/robot.urdf (robot description, URDF)
Before this commit: robot my_robot, 1 links, 0 joints
Links:
- added link link_arm, mass 0.5; collision box size=0.2 0.2 1; visual box size=0.2 0.2 1
- added link link_arm2, mass 0.5; collision box size=0.2 0.2 1; visual box size=0.2 0.2 1
- link link_chassis: mass None -> 5; geometry collision box size=1 1 2; visual box size=1 1 2
Joints:
- added joint joint1: type continuous, parent link_chassis, child link_arm, origin xyz=0.6 0 0.8 rpy=0 0 0
- added joint joint2: type continuous, parent link_chassis, child link_arm2, origin xyz=-0.6 0 0.8 rpy=0 0 0
