Commit message: tentando fazer girar

File: AmbientesRos/simulation/src/my_robot_description/urdf/braco.urdf (robot description, URDF)
Before this commit: robot braco, 3 links, 2 joints
Links:
- removed link gira_braco
- added link gira, mass 5; collision box size=0.15 0.20 0.10; visual box size=0.05 0.05 0.40
- added link testegiro, mass 5; collision box size=0.15 0.20 0.10; visual box size=0.1 0.03 0.10
Joints:
- removed joint joint2
- added joint revolute_joint: type revolute, parent base_braco, child gira, origin xyz=0 0 0.2 rpy=0 0 0, axis 0 0 1, limit lower=-1.57 upper=1.57 effort=1000 velocity=1.0
- added joint teste: type fixed, parent gira, child testegiro, origin xyz=0.03 0 0.2 rpy=0 0 0
- joint joint1: origin xyz=0.174 0 0.4 rpy=0 0 0 -> xyz=0.184 0 0.39 rpy=0 0 0
